File: idc50_breakout.kicad_pcb (KiCad board)
At the start: 2 copper layers, 17.9 x 131.7 mm, 3 parts, among them J1 Conn_01x40, J2 Conn_01x50, J3 Conn_01x10

Commit message: Updte for KiCad 6
Other:
- net class Default removed
